File: Led_cube_PCB/LED_CUBE_8x8/Layer_select.kicad_sch (KiCad schematic)
At the start: 5 parts, among them IC31 SN74HCS238DYYR, IC32 TBD62083AFNG,EL, J9 Conn_02x04_Top_Bottom

Commit message: Finalized schematic changed power source and buck converter due to unavailability stock mouser. Also assigned all the footprints to all components and ran ERC.
Parts:
- IC31: footprint SOP50P326X110-16N -> SamacSys_Parts:SOP50P326X110-16N
- IC32: footprint SOIC127P1030X245-18N -> SamacSys_Parts:SOIC127P1030X245-18N
- R59: footprint (none) -> Resistor_SMD:R_0805_2012Metric_Pad1.20x1.40mm_HandSolder
Changed lines of the file:
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@@
 			)
 		)
-		(property "Footprint" "SOP50P326X110-16N"
+		(property "Footprint" "SamacSys_Parts:SOP50P326X110-16N"
 			(at 86.36 124.13 0)
 			(hide yes)
@@
 			)
 		)
-		(property "Footprint" "SOIC127P1030X245-18N"
+		(property "Footprint" "SamacSys_Parts:SOIC127P1030X245-18N"
 			(at 87.63 177.47 0)
 			(hide yes)
@@
 			)
 		)
-		(property "Footprint" ""
+		(property "Footprint" "Resistor_SMD:R_0805_2012Metric_Pad1.20x1.40mm_HandSolder"
 			(at 40.132 45.72 90)
 			(hide yes)

Commit message: start of PCB layout
Parts:
- R59: footprint Resistor_SMD:R_0805_2012Metric_Pad1.20x1.40mm_HandSolder -> Resistor_SMD:R_0603_1608Metric_Pad0.98x0.95mm_HandSolder
Changed lines of the file:
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@@
 			)
 		)
-		(property "Footprint" "Resistor_SMD:R_0805_2012Metric_Pad1.20x1.40mm_HandSolder"
+		(property "Footprint" "Resistor_SMD:R_0603_1608Metric_Pad0.98x0.95mm_HandSolder"
 			(at 40.132 45.72 90)
 			(hide yes)
