File: Led_cube_PCB/LED_CUBE_8x8/Green_LEDS.kicad_sch (KiCad schematic)
At the start: 101 parts, among them IC1 74AHCT244PW,118, IC10 74AHCT244PW,118, IC11 74AHCT244PW,118, IC12 74AHCT244PW,118, IC2 74AHCT244PW,118, IC26 SN74HCS238DYYR, IC3 74AHCT244PW,118, IC8 74AHCT244PW,118, IC9 74AHCT244PW,118, J5 Conn_02x16_Odd_Even, J6 Conn_02x16_Odd_Even

Commit message: Finalized schematic changed power source and buck converter due to unavailability stock mouser. Also assigned all the footprints to all components and ran ERC.
Parts:
- removed TP4: TestPoint, TestPoint:TestPoint_Pad_D2.0mm, symbol Connector:TestPoint
- C1, C10, C11, C2, C3, C7, C8, C9: footprint (none) -> Capacitor_SMD:C_0805_2012Metric_Pad1.18x1.45mm_HandSolder
- IC1, IC10, IC11, IC12, IC2, IC3, IC8, IC9: footprint SOP65P640X110-20N -> SamacSys_Parts:SOP65P640X110-20N
- IC26: footprint SOP50P326X110-16N -> SamacSys_Parts:SOP50P326X110-16N
- R1, R122, R123, R124, R125, R126, R127, R128, R129, R130, R131, R132, R133, R134, R135, R136, R137, R138, R139, R140, R141, R142, R143, R144, R145, R146, R147, R148, R149, R150, R151, R152, R153, R154, R155, R156, R157, R158, R159, R160, R161, R162, R163, R164, R165, R166, R167, R168, R169, R17, R170, R171, R172, R173, R174, R175, R176, R177, R178, R179, R18, R180, R181, R182, R183, R184, R185, R19, R2, R20, R21, R22, R23, R24, R25, R4, R5, R6, R7, R8, R9: footprint (none) -> Resistor_SMD:R_0805_2012Metric_Pad1.20x1.40mm_HandSolder

Commit message: start of PCB layout
Parts:
- removed R17, R22, R23, R24, R25, R7, R8, R9: R10K, Resistor_SMD:R_0805_2012Metric_Pad1.20x1.40mm_HandSolder, symbol Device:R
- C1, C10, C11, C2, C3, C7, C8, C9: footprint Capacitor_SMD:C_0805_2012Metric_Pad1.18x1.45mm_HandSolder -> Capacitor_SMD:C_0603_1608Metric_Pad1.08x0.95mm_HandSolder
- R1, R122, R123, R124, R125, R126, R127, R128, R129, R130, R131, R132, R133, R134, R135, R136, R137, R138, R139, R140, R141, R142, R143, R144, R145, R146, R147, R148, R149, R150, R151, R152, R153, R154, R155, R156, R157, R158, R159, R160, R161, R162, R163, R164, R165, R166, R167, R168, R169, R170, R171, R172, R173, R174, R175, R176, R177, R178, R179, R18, R180, R181, R182, R183, R184, R185, R19, R2, R20, R21, R4, R5, R6: footprint Resistor_SMD:R_0805_2012Metric_Pad1.20x1.40mm_HandSolder -> Resistor_SMD:R_0603_1608Metric_Pad0.98x0.95mm_HandSolder

Commit message: Top layer placement done revised the SWD connector and started routing.
Parts:
- J5, J6: footprint Connector_PinHeader_1.00mm:PinHeader_2x16_P1.00mm_Vertical -> Connector_PinSocket_2.54mm:PinSocket_2x16_P2.54mm_Vertical
Changed lines of the file:
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@@
 			)
 		)
-		(property "Footprint" "Connector_PinHeader_1.00mm:PinHeader_2x16_P1.00mm_Vertical"
+		(property "Footprint" "Connector_PinSocket_2.54mm:PinSocket_2x16_P2.54mm_Vertical"
 			(at 335.28 152.4 0)
 			(hide yes)
@@
 			)
 		)
-		(property "Footprint" "Connector_PinHeader_1.00mm:PinHeader_2x16_P1.00mm_Vertical"
+		(property "Footprint" "Connector_PinSocket_2.54mm:PinSocket_2x16_P2.54mm_Vertical"
 			(at 335.28 101.6 0)
 			(hide yes)
