File: Led_cube_PCB/LED_CUBE_8x8/Red_LEDS.kicad_sch (KiCad schematic)
At the start: 101 parts, among them IC16 74AHCT244PW,118, IC19 74AHCT244PW,118, IC20 74AHCT244PW,118, IC21 74AHCT244PW,118, IC22 74AHCT244PW,118, IC4 74AHCT244PW,118, IC5 74AHCT244PW,118, IC6 74AHCT244PW,118, IC7 SN74HCS238DYYR, J3 Conn_02x16_Odd_Even, J4 Conn_02x16_Odd_Even

Commit message: Finalized schematic changed power source and buck converter due to unavailability stock mouser. Also assigned all the footprints to all components and ran ERC.
Parts:
- removed TP3: TestPoint, TestPoint:TestPoint_Pad_D2.0mm, symbol Connector:TestPoint
- C13, C16, C17, C18, C19, C4, C5, C6: footprint (none) -> Capacitor_SMD:C_0805_2012Metric_Pad1.18x1.45mm_HandSolder
- IC16, IC19, IC20, IC21, IC22, IC4, IC5, IC6: footprint SOP65P640X110-20N -> SamacSys_Parts:SOP65P640X110-20N
- IC7: footprint SOP50P326X110-16N -> SamacSys_Parts:SOP50P326X110-16N
- R10, R100, R101, R102, R103, R104, R105, R106, R107, R108, R109, R11, R110, R111, R112, R113, R114, R115, R116, R117, R118, R119, R12, R120, R121, R13, R14, R15, R16, R31, R32, R37, R38, R39, R40, R41, R42, R43, R44, R60, R61, R62, R63, R64, R65, R66, R67, R68, R69, R70, R71, R72, R73, R74, R75, R76, R77, R78, R79, R80, R81, R82, R83, R84, R85, R86, R87, R88, R89, R90, R91, R92, R93, R94, R95, R96, R97, R98, R99: footprint (none) -> Resistor_SMD:R_0805_2012Metric_Pad1.20x1.40mm_HandSolder
- R52, R53: renamed from R; footprint (none) -> Resistor_SMD:R_0805_2012Metric_Pad1.20x1.40mm_HandSolder

Commit message: start of PCB layout
Parts:
- removed R14, R15, R16, R32, R41, R42, R43, R44: R10K, Resistor_SMD:R_0805_2012Metric_Pad1.20x1.40mm_HandSolder, symbol Device:R
- C13, C16, C17, C18, C19, C4, C5, C6: footprint Capacitor_SMD:C_0805_2012Metric_Pad1.18x1.45mm_HandSolder -> Capacitor_SMD:C_0603_1608Metric_Pad1.08x0.95mm_HandSolder
- R10, R100, R101, R102, R103, R104, R105, R106, R107, R108, R109, R11, R110, R111, R112, R113, R114, R115, R116, R117, R118, R119, R12, R120, R121, R13, R31, R37, R38, R39, R40, R52, R53, R60, R61, R62, R63, R64, R65, R66, R67, R68, R69, R70, R71, R72, R73, R74, R75, R76, R77, R78, R79, R80, R81, R82, R83, R84, R85, R86, R87, R88, R89, R90, R91, R92, R93, R94, R95, R96, R97, R98, R99: footprint Resistor_SMD:R_0805_2012Metric_Pad1.20x1.40mm_HandSolder -> Resistor_SMD:R_0603_1608Metric_Pad0.98x0.95mm_HandSolder

Commit message: Top layer placement done revised the SWD connector and started routing.
Parts:
- J3, J4: footprint Connector_PinHeader_1.00mm:PinHeader_2x16_P1.00mm_Vertical -> Connector_PinSocket_2.54mm:PinSocket_2x16_P2.54mm_Vertical
Changed lines of the file:
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@@
 			)
 		)
-		(property "Footprint" "Connector_PinHeader_1.00mm:PinHeader_2x16_P1.00mm_Vertical"
+		(property "Footprint" "Connector_PinSocket_2.54mm:PinSocket_2x16_P2.54mm_Vertical"
 			(at 335.28 110.49 0)
 			(hide yes)
@@
 			)
 		)
-		(property "Footprint" "Connector_PinHeader_1.00mm:PinHeader_2x16_P1.00mm_Vertical"
+		(property "Footprint" "Connector_PinSocket_2.54mm:PinSocket_2x16_P2.54mm_Vertical"
 			(at 335.28 161.29 0)
 			(hide yes)
